File: pcb/starman.kicad_sch (KiCad schematic)
At the start: 220 parts, among them J1 M20-8771246, J2 M20-8771246, J3 M20-8771246, U1 ESP32-S3-MINI-1, U10 LED1642GWTTR, U11 AZ1084CS2-ADJ, U12 BA33BC0FP-E2, U2 LED1642GWTTR, U3 LED1642GWTTR, U4 LED1642GWTTR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

Commit message: Bump the variable resistor to 20k, update the schematics, BOM for printing
Also marked C33 & D145 as NC (never could get it to work). It should
be replaced by a proper multi-lead RGB LED
Parts:
- C33: value 1uF -> 1uF nc
- D145: value WS2812B -> WS2812B nc
Other:
- moved on the sheet: C1, C10, C11, C12, C13, C14, C15, C16, C17, C18, C19, C2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
